File: PCB_NCV-ShakeIt/NCV-ShakeIt/_autosave-NCV-ShakeIt.kicad_pcb (KiCad board)
At the start: 2 copper layers, 55 x 47 mm, 15 parts, among them U1 XIAO-SAMD21-DIP, U2 DFR0299

Commit message: Adding to docs, fixing code, renaming things to be more clear
Parts:
- added Override1: Conn_01x02_Pin, Connector_PinHeader_2.54mm:PinHeader_1x02_P2.54mm_Vertical, F.Cu at (26.0, 63.5)
- moved POT_SENSITIVITY1 2.00 mm to (39.0, 63.5)
Connections:
- SPK1 pad 1: GND -> Net-(U2-SPK2)
- U1 pad 1: unconnected-(U1-PA02_A0_D0-Pad1) -> Net-(OverrideSwitch1-Pin_2)
- U2 pad 8: unconnected-(U2-SPK2-Pad8) -> Net-(U2-SPK2)
Routing:
- net Net-(OverrideSwitch1-Pin_2): track 0.00 -> 60.3 mm, vias 0 -> 1
- net Net-(U2-SPK2): track 0.00 -> 16.1 mm
- net GND: track 154.5 -> 148.7 mm
- net Net-(U1-PA7_A8_D8_SCK): track 24.7 -> 30.3 mm
- net +5V: track 89.8 -> 91.9 mm
- net +3.3V: track 86.4 -> 88.4 mm
- net Net-(GREEN_EMF1-K): track 23.3 -> 22.4 mm
Other:
- board text added: "NCV-ShakeIt V2 by Jon Garrison jongarrison.github.io"
- board text removed: "NCV-ShakeIt by Jon Garrison jongarrison.github.io"
